File: WolfNet-65816-GPC.kicad_sch (KiCad schematic)
At the start: 38 parts, among them J1 ATX-24, SW1 SW_SPST, SW2 SW_Push, U1 WD65C816S, U10 DS1813, U2 74HCT573, U3 74HCT245, U4 AS6C1608, U5 XCR3064XL-VQ100, U6 28C040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

Commit message: Update WolfNet-65816-GPC.kicad_sch
Parts:
- removed U6, U7: 28C040, symbol Memory:28C040
- added U8: SST39SF040, symbol Memory_Flash:SST39SF040
- X2: renamed from X?; value ACO-xxxMHz -> ACO-3.6864MHz
- gave numbers to parts that had none: 25
- renumbered J1 to J6, U10 to U12, U2 to U3, U3 to U4, U4 to U5, U5 to U6
Connections:
- net A0: now also U8.12 (A0)
- net A1: now also U8.11 (A1)
- net A10: now also U7.23 (A10), U8.23 (A10)
- net A11: now also U7.25 (A11), U8.25 (A11)
- net A12: now also U7.4 (A12), U8.4 (A12)
- net A13: now also U7.28 (A13), U8.28 (A13)
- net A14: now also U7.29 (A14), U8.29 (A14)
- net A15: now also U7.3 (A15), U8.3 (A15)
- net A16: now also U7.2 (A16), U8.2 (A16)
- net A17: now also U7.30 (A17), U8.30 (A17)
- net A18: now also U7.1 (A18), U8.1 (A18)
- net A2: now also U8.10 (A2)
- net A3: now also U8.9 (A3)
- net A4: now also U7.8 (A4), U8.8 (A4)
- net A5: now also U7.7 (A5), U8.7 (A5)
- net A6: now also U7.6 (A6), U8.6 (A6)
- net A7: now also U7.5 (A7), U8.5 (A7)
- net A8: now also U7.27 (A8), U8.27 (A8)
- net A9: now also U7.26 (A9), U8.26 (A9)
- net D0: now also U8.13 (D0)
- net D1: now also U8.14 (D1)
- net D2: now also U8.15 (D2)
- net D3: now also U8.17 (D3)
- net D4: now also U8.18 (D4)
- net D5: now also U8.19 (D5)
- net D6: now also U8.20 (D6)
- net D7: now also U8.21 (D7)
- net GND: now also U8.16 (GND)
- net R/~{W}: now also U8.31 (PGM)
- net VCC: now also U8.32 (VCC)
- net ~{FLASH_EN}: now also U8.22 (CE)
- net ~{FLASH_OE}: now also U8.24 (OE)
Other:
- moved on the sheet: U7, X2

Commit message: Update WolfNet-65816-GPC.kicad_sch
Connections:
- net ~{FLASH_EN} renamed ~{FLASH1_EN}
- net ~{FLASH1_EN}: no longer U8.22 (CE)
- net ~{FLASH_OE} renamed ~{FLASH1_OE}
- net ~{FLASH1_OE}: no longer U8.24 (OE)
- new net ~{FLASH2_EN}: U8.22 (CE)
- new net ~{FLASH2_OE}: U8.24 (OE)
Changed lines of the file:
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@@
     )
   )
-  (global_label "~{FLASH_EN}" (shape input) (at 218.44 78.74 180) (fields_autoplaced)
-    (effects (font (size 1.27 1.27)) (justify right))
-    (property "Intersheet References" "${INTERSHEET_REFS}" (id 0) (at 206.8345 78.6606 0)
+  (global_label "~{FLASH2_EN}" (shape input) (at 218.44 78.74 180) (fields_autoplaced)
+    (effects (font (size 1.27 1.27)) (justify right))
+    (property "Intersheet References" "${INTERSHEET_REFS}" (id 0) (at 205.625 78.6606 0)
       (effects (font (size 1.27 1.27)) (justify right) hide)
     )
@@
     )
   )
-  (global_label "~{FLASH_EN}" (shape input) (at 176.53 78.74 180) (fields_autoplaced)
-    (effects (font (size 1.27 1.27)) (justify right))
-    (property "Intersheet References" "${INTERSHEET_REFS}" (id 0) (at 164.9245 78.6606 0)
+  (global_label "~{FLASH1_EN}" (shape input) (at 176.53 78.74 180) (fields_autoplaced)
+    (effects (font (size 1.27 1.27)) (justify right))
+    (property "Intersheet References" "${INTERSHEET_REFS}" (id 0) (at 163.715 78.6606 0)
       (effects (font (size 1.27 1.27)) (justify right) hide)
     )
@@
     )
   )
-  (global_label "~{FLASH_OE}" (shape input) (at 176.53 81.28 180) (fields_autoplaced)
-    (effects (font (size 1.27 1.27)) (justify right))
-    (property "Intersheet References" "${INTERSHEET_REFS}" (id 0) (at 164.9245 81.2006 0)
+  (global_label "~{FLASH1_OE}" (shape input) (at 176.53 81.28 180) (fields_autoplaced)
+    (effects (font (size 1.27 1.27)) (justify right))
+    (property "Intersheet References" "${INTERSHEET_REFS}" (id 0) (at 163.715 81.2006 0)
       (effects (font (size 1.27 1.27)) (justify right) hide)
     )
@@
     )
   )
-  (global_label "~{FLASH_OE}" (shape input) (at 218.44 81.28 180) (fields_autoplaced)
-    (effects (font (size 1.27 1.27)) (justify right))
-    (property "Intersheet References" "${INTERSHEET_REFS}" (id 0) (at 206.8345 81.2006 0)
-      (effects (font (size 1.27 1.27)) (justify right) hide)
-    )
+  (global_label "~{FLASH2_OE}" (shape input) (at 218.44 81.28 180) (fields_autoplaced)
+    (effects (font (size 1.27 1.27)) (justify right))
+    (property "Intersheet References" "${INTERSHEET_REFS}" (id 0) (at 205.625 81.2006 0)
+      (effects (font (size 1.27 1.27)) (justify right) hide)
+    )
