File: WolfNet-65816-GPC.kicad_sch (KiCad schematic)
At the start: 37 parts, among them J1 Conn_01x01, J2 Conn_01x01, J3 Conn_01x01, J4 Conn_01x01, J5 USB_B, J6 ATX-24, SW1 SW_SPST, SW2 SW_Push, U1 WD65C816S, U10 LM7905_TO220, U11 SC28L91, U12 DS1813, U2 MCP2200-I-SO, U3 74HCT573, U4 74HCT245, U5 AS6C1608, U6 XCR3064XL-VQ100, U7 SST39SF040, U8 SST39SF040, U9 XCR3064XL-VQ100, X1 ACO-12MHz, X2 ACO-3.6864MHz

Commit message: Update WolfNet-65816-GPC.kicad_sch
Connections:
- net ~{RESET}: no longer U11.38 (RESET)
- new net RESET: U11.38 (RESET)
Changed lines of the file:
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@@
     )
   )
-  (global_label "~{RESET}" (shape input) (at 378.46 39.37 0) (fields_autoplaced)
+  (global_label "RESET" (shape input) (at 378.46 39.37 0) (fields_autoplaced)
     (effects (font (size 1.27 1.27)) (justify left))
     (property "Intersheet References" "${INTERSHEET_REFS}" (id 0) (at 386.6183 39.2906 0)

Commit message: Update WolfNet-65816-GPC.kicad_sch
Parts:
- added U?: WD65C22, symbol 65xx:WD65C22
Other:
- note added: "Connectors"
Changed lines of the file:
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@@
     (effects (font (size 1.27 1.27)) (justify left bottom))
   )
+  (text "Connectors" (at 104.14 213.36 0)
+    (effects (font (size 1.27 1.27)) (justify left bottom))
+  )
   (text "UART" (at 326.39 20.32 0)
     (effects (font (size 1.27 1.27)) (justify left bottom))
@@
     (pin "1")
   )
+  (symbol (lib_id "65xx:WD65C22") (at 290.83 48.26 0) (unit 1)
+    (in_bom yes) (on_board yes) (fields_autoplaced)
+    (property "Reference" "U?" (id 0) (at 290.83 17.78 0)
+      (effects (font (size 1.524 1.524)))
+    )
+    (property "Value" "WD65C22" (id 1) (at 290.83 21.59 0)
+      (effects (font (size 1.524 1.524)))
+    )
+    (property "Footprint" "" (id 2) (at 278.13 43.18 0)
+      (effects (font (size 1.524 1.524)))
+    )
+    (property "Datasheet" "" (id 3) (at 278.13 43.18 0)
+      (effects (font (size 1.524 1.524)))
+    )
+    (pin "1")
+    (pin "10")
+    (pin "11")
+    (pin "12")
+    (pin "13")
+    (pin "14")
+    (pin "15")
+    (pin "16")
+    (pin "17")
+    (pin "18")
+    (pin "19")
+    (pin "2")
+    (pin "20")
+    (pin "21")
+    (pin "22")
+    (pin "23")
+    (pin "24")
+    (pin "25")
+    (pin "26")
+    (pin "27")
+    (pin "28")
+    (pin "29")
+    (pin "3")
+    (pin "30")
+    (pin "31")
+    (pin "32")
+    (pin "33")
+    (pin "34")
+    (pin "35")
+    (pin "36")
+    (pin "37")
+    (pin "38")
+    (pin "39")
+    (pin "4")
+    (pin "40")
+    (pin "5")
+    (pin "6")
+    (pin "7")
+    (pin "8")
+    (pin "9")
+  )
   (symbol (lib_id "Connector_Generic:Conn_01x01") (at 284.48 88.9 90) (unit 1)
     (in_bom yes) (on_board yes)
@@
       (reference "U12") (unit 1) (value "DS1813") (footprint "")
     )
+    (path "/df343ba5-b168-47a5-aec0-32979ea9c319"
+      (reference "U?") (unit 1) (value "WD65C22") (footprint "")
+    )
     (path "/3cdba75b-c996-41f4-b832-36b346107ba1"

Commit message: Update WolfNet-65816-GPC.kicad_sch
Parts:
- removed U6: XCR3064XL-VQ100, Package_QFP:LQFP-100_14x14mm_P0.5mm, symbol CPLD_Xilinx:XCR3064XL-VQ100
- added J?: 65SIB_Connector, symbol Connector (Open HW):65SIB_Connector
- added U?: XCR3256XL-TQ144, Package_QFP:TQFP-144_20x20mm_P0.5mm, symbol CPLD_Xilinx:XCR3256XL-TQ144
- added U?: 74HCT137, symbol 74xx:74HCT137
- added U?: 28C16, symbol Memory:28C16
Connections:
- net +12V: now also J?.10 (12v), J?.8 (12v)
- net +5V: now also U?.20 (VCC), U?.115 (VCC), U?.123 (VCC), U?.130 (VCC), U?.144 (VCC), U?.16 (VCC), U?.24 (VCC), U?.24 (VCC), U?.50 (VCC), U?.51 (VCC), U?.58 (VCC), U?.73 (VCC), U?.76 (VCC), U?.95 (VCC)
- net -12V: now also J?.13 (-12v)
- net A0: now also U?.38 (RS0), U?.8 (A0)
- net A1: now also U?.37 (RS1), U?.7 (A1)
- net A10: now also U?.19 (A10)
- net A2: now also U?.36 (RS2), U?.6 (A2)
- net A3: now also U?.35 (RS3), U?.5 (A3)
- net A4: now also U?.4 (A4)
- net A5: now also U?.3 (A5)
- net A6: now also U?.2 (A6)
- net A7: now also U?.1 (A7)
- net A8: now also U?.23 (A8)
- net A9: now also U?.22 (A9)
- net D0: now also U?.33 (D0), U?.9 (D0)
- net D1: now also U?.32 (D1), U?.10 (D1)
- net D2: now also U?.31 (D2), U?.11 (D2)
- net D3: now also U?.30 (D3), U?.13 (D3)
- net D4: now also U?.29 (D4), U?.14 (D4)
- net D5: now also U?.28 (D5), U?.15 (D5)
- net D6: now also U?.27 (D6), U?.16 (D6)
- net D7: now also U?.26 (D7), U?.17 (D7)
- net DMA_JTAG: now also U?.13 (PORT_EN)
- net GND: now also U?.1 (GND), J?.16 (GND), J?.19 (GND), J?.2 (GND), J?.4 (GND), J?.6 (eGND), U?.105 (GND), U?.12 (GND), U?.124 (GND), U?.129 (GND), U?.135 (GND), U?.17 (GND), U?.3 (GND), U?.33 (GND), U?.52 (GND), U?.57 (GND), U?.59 (GND), U?.64 (GND), U?.8 (GND), U?.85 (GND)
- net PHI2: now also U?.25 (PHI2), U?.128 (CLK0/IN0)
- net RESET: now also J2.1 (Pin_1), U9.62 (C0/TCK)
- net R/~{W}: now also U?.22 (R/~{W})
- net ~{IRQ}: no longer JP1.1 (A)
- net ~{READ}: now also U?.20 (~{OE})
- net ~{RESET}: now also U?.34 (~{RESET})
- net ~{WRITE}: now also U?.21 (~{WE})
- net ~{E_ROM_CS}: now reaches U9.21 (D5)
- net ~{E_ROM_CS}: now also U?.18 (~{CS})
- net ~{C22_CS2}: now reaches U9.23 (D6)
- net ~{C22_CS2}: now also U?.23 (~{CS2}), U?.5 (~{E1})
- net C22_CS1: now reaches U9.25 (D7)
- net C22_CS1: now also U?.24 (CS1), U?.6 (E2)
- net ~{65SIB_IRQ}: now reaches U9.88 (CLK2/IN2)
- net ~{65SIB_IRQ}: now also U?.21 (~{IRQ})
- net ~{UART_IRQ}: now reaches U9.89 (CLK1/IN1)
- net ~{UART_IRQ}: now also JP1.1 (A)
- net PA0: now reaches U?.2 (PA0)
- net PA1: now reaches U?.3 (PA1)
- net PA2: now reaches U?.4 (PA2)
- net ~{C22_IRQ1}: now reaches U?.40 (CA1)
- net ~{C22_IRQ1}: now also J?.9 (IRO\)
- net PA3: now reaches U?.5 (PA3)
- net ~{CONF}: now reaches U?.6 (PA4)
- net ~{CONF}: now also J?.1 (CONF\)
- net 65SIB_MOSI: now reaches U?.7 (PA5)
- net 65SIB_MOSI: now also J?.5 (MOSI)
- net 65SIB_MISO: now reaches U?.8 (PA6)
- net 65SIB_MISO: now also J?.7 (MISO)
- net 65SIB_CLK: now reaches U?.9 (PA7)
- net 65SIB_CLK: now also J?.3 (CLK)
- new net PB0: U?.1 (A0)
- new net PB1: U?.2 (A1)
- new net PB2: U?.3 (A2)
- new net PB3: U?.4 (~{LE})
- new net ~{SEL1}: J?.11 (SEL1\), U?.14 (~{Y1})
- new net ~{SEL2}: J?.12 (SEL2\), U?.13 (~{Y2})
- new net ~{SEL3}: J?.14 (SEL3\), U?.12 (~{Y3})
- new net ~{SEL4}: J?.15 (SEL4\), U?.11 (~{Y4})
- new net ~{SEL5}: J?.17 (SEL5\), U?.10 (~{Y5})
- new net ~{SEL6}: J?.18 (SEL6\), U?.9 (~{Y6})
- new net ~{SEL7}: J?.20 (SEL7\), U?.7 (~{Y7})
- no-connect marks 38 -> 39
Other:
- note added: "65C02 Compatibility"
- note added: "65SIB"
- note added: "DMA Controller"
- note removed: "Connectors"
- note removed: "Direct Memory Access Circuit"
- moved on the sheet: J1, J2, J3, R2, R3, R4, U1, U?, X2

Commit message: Update WolfNet-65816-GPC.kicad_sch
Parts:
- added J? (x2): Bus_ISA_8bit, symbol Connector:Bus_ISA_8bit
Connections:
- net +12V: now also J?.9 (+12V)
- net +5V: now also J?.3 (VCC)
- net -12V: now also J?.7 (-12V)
- net -5V: now also J?.5 (-5V)
- net GND: now also J?.1 (GND), J?.10 (GND), J?.31 (GND)
Other:
- moved on the sheet: U3, U4, U?

Commit message: Update WolfNet-65816-GPC.kicad_sch
Parts:
- removed U?: XCR3256XL-TQ144, Package_QFP:TQFP-144_20x20mm_P0.5mm, symbol CPLD_Xilinx:XCR3256XL-TQ144
- removed X1: ACO-12MHz, Oscillator:Oscillator_DIP-14, symbol Oscillator:ACO-xxxMHz
- added J? (x4): Conn_01x01, symbol Connector_Generic:Conn_01x01
- added U?: XCR3064-VQ100, Package_QFP:LQFP-100_14x14mm_P0.5mm, symbol CPLD_Xilinx:XCR3064-VQ100
- added U?: 74HCT163, symbol 74xx:74LS163
- added X?: ACO-24MHz, Oscillator:Oscillator_DIP-14, symbol Oscillator:ACO-xxxMHz
Connections:
- net +12V: now also J?.9 (+12V)
- net +5V: now also J?.29 (VCC), J?.3 (VCC), U?.1 (~{MR}), U?.10 (CET), U?.16 (VCC), U?.18 (VCC), U?.3 (VCC), U?.34 (VCC), U?.39 (VCC), U?.51 (VCC), U?.66 (VCC), U?.7 (CEP), U?.82 (VCC), U?.91 (VCC), X?.14 (Vcc)
- net -12V: now also J?.7 (-12V)
- net -5V: now also J?.5 (-5V)
- net A0: now also J?.62 (BA00), J?.62 (BA00)
- net A1: now also J?.61 (BA01), J?.61 (BA01)
- net A10: now also J?.52 (BA10), J?.52 (BA10)
- net A11: now also J?.51 (BA11), J?.51 (BA11)
- net A12: now also J?.50 (BA12), J?.50 (BA12)
- net A13: now also J?.49 (BA13), J?.49 (BA13)
- net A14: now also J?.48 (BA14), J?.48 (BA14)
- net A15: now also J?.47 (BA15), J?.47 (BA15)
- net A16: now also J?.46 (BA16), J?.46 (BA16)
- net A17: now also J?.45 (BA17), J?.45 (BA17)
- net A18: now also J?.44 (BA18), J?.44 (BA18)
- net A19: now also J?.43 (BA19), J?.43 (BA19)
- net A2: now also J?.60 (BA02), J?.60 (BA02)
- net A3: now also J?.59 (BA03), J?.59 (BA03)
- net A4: now also J?.58 (BA04), J?.58 (BA04)
- net A5: now also J?.57 (BA05), J?.57 (BA05)
- net A6: now also J?.56 (BA06), J?.56 (BA06)
- net A7: now also J?.55 (BA07), J?.55 (BA07)
- net A8: now also J?.54 (BA08), J?.54 (BA08)
- net A9: now also J?.53 (BA09), J?.53 (BA09)
- net BusEnable: now also J?.42 (AEN), J?.42 (AEN)
- net D0: now also J?.40 (DB0), J?.40 (DB0)
- net D1: now also J?.39 (DB1), J?.39 (DB1)
- net D2: now also J?.38 (DB2), J?.38 (DB2)
- net D3: now also J?.37 (DB3), J?.37 (DB3)
- net D4: now also J?.36 (DB4), J?.36 (DB4)
- net D5: now also J?.35 (DB5), J?.35 (DB5)
- net D6: now also J?.34 (DB6), J?.34 (DB6)
- net D7: now also J?.33 (DB7), J?.33 (DB7)
- net DMA_JTAG: now also U?.11 (PORT_EN)
- net GND: now also J?.1 (GND), J?.10 (GND), J?.31 (GND), U?.26 (GND), U?.38 (GND), U?.43 (GND), U?.59 (GND), U?.74 (GND), U?.8 (GND), U?.86 (GND), U?.95 (GND), X?.7 (GND)
- net PHI2: now also J?.20 (CLK), J?.20 (CLK), U?.90 (CLK0/IN0)
- net RDY: now also U?.85 (A0)
- net RESET: now also J?.2 (RESET), J?.2 (RESET), U?.89 (CLK1/IN1)
- net CLK0: now reaches U2.2 (OSC1)
- net CLK0: now also U?.14 (Q0)
- net IRQ: now reaches J?.21 (IRQ7)
- net IRQ: now also J?.22 (IRQ6), J?.23 (IRQ5), J?.24 (IRQ4), J?.25 (IRQ3), J?.4 (IRQ2)
- net CLOCK renamed CLK1
- net CLK1: now also U?.11 (Q3), U?.9 (~{PE})
- new net: J?.1 (Pin_1), U?.15 (D0/TMS)
- new net: J?.1 (Pin_1), U?.4 (B8/TDI)
- new net: J?.1 (Pin_1), U?.62 (C0/TCK)
- new net: J?.1 (Pin_1), U?.73 (A8/TDO)
- new net: U?.2 (CP), X?.8 (OUT)
- no-connect marks 39 -> 54
Other:
- note added: "65C02 Compatibility ROM"
- note removed: "65C02 Compatibility"
- moved on the sheet: J?

Commit message: Connected ISA ports...
Parts:
- removed U?: 28C16, symbol Memory:28C16
- removed X?: ACO-24MHz, Oscillator:Oscillator_DIP-14, symbol Oscillator:ACO-xxxMHz
- added D2: D, Diode_THT:D_A-405_P7.62mm_Horizontal, symbol Device:D
- added R6, R7, R8, R9: 3.3k, symbol Device:R
- added X2: ACO-24MHz, Oscillator:Oscillator_DIP-14, symbol Oscillator:ACO-xxxMHz
- added X3: ACO-14.31818MHz, Oscillator:Oscillator_DIP-14, symbol Oscillator:ACO-xxxMHz
- C1: renamed from C4; footprint (none) -> Capacitor_THT:CP_Radial_D5.0mm_P2.50mm
- C2: renamed from C1; footprint (none) -> Capacitor_THT:CP_Radial_D5.0mm_P2.50mm
- C3: renamed from C2; footprint (none) -> Capacitor_THT:C_Disc_D3.8mm_W2.6mm_P2.50mm
- C4: renamed from C3; footprint (none) -> Capacitor_THT:C_Disc_D3.8mm_W2.6mm_P2.50mm
- D1: renamed from D3; footprint (none) -> LED_THT:LED_D3.0mm
- D3: renamed from D1; footprint (none) -> LED_THT:LED_D3.0mm
- D4: renamed from D2; footprint (none) -> LED_THT:LED_D3.0mm
- J1: renamed from J3; footprint (none) -> Connector_Pin:Pin_D1.0mm_L10.0mm
- J11: renamed from J5; footprint (none) -> Connector_USB:USB_Mini-B_Tensility_54-00023_Vertical; symbol Connector:USB_B -> Connector:USB_B_Mini
- J2: renamed from J1; footprint (none) -> Connector_Pin:Pin_D1.0mm_L10.0mm
- J3: renamed from J2; footprint (none) -> Connector_Pin:Pin_D1.0mm_L10.0mm
- J4: footprint (none) -> Connector_Pin:Pin_D1.0mm_L10.0mm
- J5, J6, J7, J8: renamed from J?; footprint (none) -> Connector_Pin:Pin_D1.0mm_L10.0mm
- gave numbers to parts that had none: 7
- renumbered J6 to J10, R2 to R1, R1 to R10, R5 to R11, R3 to R2, R4 to R3, R6 to R4, R7 to R5, SW2 to SW1, SW1 to SW2, U11 to U1, U9 to U10, U10 to U12, U2 to U13, U5 to U2, U7 to U4, U8 to U5, U1 to U6, U12 to U7, U4 to U8, U3 to U9, X2 to X1
Connections:
- net +5V: now also J12.29 (VCC), X2.14 (Vcc), X3.14 (Vcc)
- net CLK1: no longer U14.11 (Q3), U14.9 (~{PE})
- net GND: now also J11.6 (Shield), D2.1 (K), X2.7 (GND), X3.7 (GND); no longer J11.4 (GND)
- net IRQ: now also J12.21 (IRQ7), J12.22 (IRQ6), J12.23 (IRQ5), J12.24 (IRQ4), J12.25 (IRQ3), J12.4 (IRQ2)
- net PHI2: no longer J12.20 (CLK), J9.20 (CLK), U10.90 (CLK0/IN0)
- net RDY: now also J7.1 (Pin_1), U11.62 (C0/TCK), U11.88 (CLK2/IN2); no longer U11.85 (A0)
- net ~{IRQ}: now also U10.40 (C15)
- net ~{READ}: now also U10.47 (C9); no longer U10.12 (B13)
- net ~{WRITE}: now also U10.46 (C10); no longer U10.13 (B14)
- net ~{SMEMW}: now reaches J12.11 (~{SMEMW})
- net ~{SMEMW}: now also J9.11 (~{SMEMW}), U10.41 (C14)
- net ~{SMEMR}: now reaches J12.12 (~{SMEMR})
- net ~{SMEMR}: now also J9.12 (~{SMEMR}), U10.42 (C13)
- net ~{IOW}: now reaches J12.13 (~{IOW})
- net ~{IOW}: now also J9.13 (~{IOW}), U10.44 (C12)
- net ~{IOR}: now reaches J12.14 (~{IOR})
- net ~{IOR}: now also J9.14 (~{IOR}), U10.45 (C11)
- net ~{DACK3}: now reaches J12.15 (~{DACK3})
- net ~{DACK3}: now also J9.15 (~{DACK3})
- net ~{DRQ3}: now reaches J12.16 (DRQ3)
- net ~{DRQ3}: now also J9.16 (DRQ3), J9.18 (DRQ1)
- net ~{DACK1}: now reaches J12.17 (~{DACK1})
- net ~{DACK1}: now also J9.17 (~{DACK1})
- net ~{DRQ1}: now reaches J12.18 (DRQ1)
- net ~{DACK0}: now reaches J12.19 (~{DACK0})
- net ~{DACK0}: now also J9.19 (~{DACK0})
- net ~{DACK2}: now reaches J12.26 (~{DACK2})
- net ~{DACK2}: now also J9.26 (~{DACK2})
- net T/C: now reaches J12.27 (TC)
- net T/C: now also J8.1 (Pin_1), J9.27 (TC), U11.73 (A8/TDO)
- net LATCH_EN: now reaches J12.28 (ALE)
- net LATCH_EN: now also J9.28 (ALE)
- net ISA_CLK: now reaches J12.30 (OSC)
- net ISA_CLK: now also J9.30 (OSC), X3.8 (OUT)
- net IO_CHK1: now reaches J12.32 (IO)
- net IO_RDY: now reaches J12.41 (IO_READY)
- net IO_RDY: now also J9.41 (IO_READY)
- net ~{DRQ2}: now reaches J12.6 (DRQ2)
- net ~{DRQ2}: now also J9.6 (DRQ2)
- net ~{HALT}: now reaches J1.1 (Pin_1), U10.15 (D0/TMS)
- net ~{HALT}: now also R6.1, R7.1, R8.1, R9.1
- net IO_CHK0: now reaches J9.32 (IO)
- net CLK_STR: now reaches U14.12 (Q2)
- net CLK_STR: now also J12.20 (CLK), J9.20 (CLK)
- net at U14.2 (CP): now also X2.8 (OUT)
- net at U14.3 (D0): now also R9.2
- net at U14.4 (D1): now also R8.2
- net at U14.5 (D2): now also D2.2 (A), R7.2
- net at U14.6 (D3): now also R6.2
- net CLK0 renamed CLK_STD
- net CLK_STD: now also U10.90 (CLK0/IN0)
- net ~{E_ROM_CS}: no longer names the net of U10.21 (D5)
- new net: U14.11 (Q3), U14.9 (~{PE})
Other:
- note added: "65SIB Controller"
- note added: "Clock Stretcher"
- note added: "ISA Buses"
- note removed: "65C02 Compatibility ROM"
- moved on the sheet: J5, J6, J7, J8, SW1, U11, U14, U15, U7
