File: Motherboard/Motherboard.kicad_pcb (KiCad board)
At the start: 4 copper layers, 246.4 x 175.3 mm, 56 parts, among them J1 40-pin IDE Connector, J3 Bus_ISA_8bit, J4 ATX-24, J5 USB_B, J6 ATF15XX_JTAG_ISP, J7 Bus_ISA_8bit, J8 65SIB_Connector, SW1 SW_Push, SW2 SW_SPST, U1 AS6C8008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

Commit message: 305 unrouted traces...
Routing:
- net GND: track 1167.0 -> 1222.1 mm, vias 2 -> 4
Changed lines of the file:
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@@
   (segment (start 315.235 73.945) (end 315.235 83.245) (width 0.25) (layer "F.Cu") (net 2))
   (segment (start 165.260374 215.963) (end 164.6438 215.963) (width 0.25) (layer "F.Cu") (net 2))
+  (segment (start 276.3698 72.7532) (end 276.352 72.771) (width 0.25) (layer "F.Cu") (net 2))
   (segment (start 175.253026 193.3326) (end 175.8696 193.3326) (width 0.25) (layer "F.Cu") (net 2))
+  (segment (start 281.9908 72.7532) (end 276.3698 72.7532) (width 0.25) (layer "F.Cu") (net 2))
   (segment (start 284.3658 83.7532) (end 283.2408 82.6282) (width 0.25) (layer "F.Cu") (net 2))
   (segment (start 315.81 68.82) (end 315.034 69.596) (width 0.25) (layer "F.Cu") (net 2))
@@
   (segment (start 225.63 83.185) (end 223.266 83.185) (width 0.25) (layer "F.Cu") (net 2))
   (segment (start 175.8188 215.163) (end 170.561 215.163) (width 0.25) (layer "F.Cu") (net 2))
+  (segment (start 164.6438 215.963) (end 152.717 215.963) (width 0.25) (layer "F.Cu") (net 2))
   (segment (start 282.8158 72.7532) (end 283.7908 71.7782) (width 0.25) (layer "F.Cu") (net 2))
   (segment (start 170.561 215.163) (end 166.060374 215.163) (width 0.25) (layer "F.Cu") (net 2))
@@
   (segment (start 88.4174 180.1876) (end 100.3046 180.1876) (width 0.25) (layer "F.Cu") (net 2))
   (segment (start 100.3046 180.1876) (end 102.23 178.2622) (width 0.25) (layer "F.Cu") (net 2))
+  (segment (start 152.717 215.963) (end 152.654 215.9) (width 0.25) (layer "F.Cu") (net 2))
   (segment (start 170.307 194.1326) (end 170.307 215.163) (width 0.25) (layer "F.Cu") (net 2))
+  (via (at 152.654 215.9) (size 0.8) (drill 0.4) (layers "F.Cu" "B.Cu") (net 2))
   (via (at 223.2152 83.1342) (size 0.8) (drill 0.4) (layers "F.Cu" "B.Cu") (net 2))
+  (via (at 276.352 72.771) (size 0.8) (drill 0.4) (layers "F.Cu" "B.Cu") (net 2))
   (via (at 225.6028 77.6732) (size 0.8) (drill 0.4) (layers "F.Cu" "B.Cu") (net 2))
   (segment (start 235.5166 65.8254) (end 235.5166 79.966) (width 0.25) (layer "B.Cu") (net 2))
@@
   (segment (start 98.6028 88.773) (end 98.6028 96.52) (width 0.25) (layer "B.Cu") (net 2))
   (segment (start 167.6654 96.2406) (end 167.6654 100.965) (width 0.25) (layer "B.Cu") (net 2))
+  (segment (start 264.9366 72.771) (end 257.683 80.0246) (width 0.25) (layer "B.Cu") (net 2))
+  (segment (start 138.793 215.283) (end 137.668 216.408) (width 0.25) (layer "B.Cu") (net 2))
   (segment (start 117.38 82.435) (end 117.38 96.4372) (width 0.25) (layer "B.Cu") (net 2))
   (segment (start 314.0644 184.499) (end 314.1472 184.5818) (width 0.25) (layer "B.Cu") (net 2))
@@
   (segment (start 222.0162 110.8254) (end 222.0162 131.0438) (width 0.25) (layer "B.Cu") (net 2))
   (segment (start 209.7838 133.1162) (end 209.7838 131.0438) (width 0.25) (layer "B.Cu") (net 2))
+  (segment (start 152.654 215.9) (end 152.037 215.283) (width 0.25) (layer "B.Cu") (net 2))
   (segment (start 106.426 96.52) (end 101.6 96.52) (width 0.25) (layer "B.Cu") (net 2))
   (segment (start 242.8748 80.0246) (end 240.792 80.0246) (width 0.25) (layer "B.Cu") (net 2))
+  (segment (start 276.352 72.771) (end 264.9366 72.771) (width 0.25) (layer "B.Cu") (net 2))
   (segment (start 98.6028 96.52) (end 101.6 96.52) (width 0.25) (layer "B.Cu") (net 2))
+  (segment (start 152.037 215.283) (end 138.793 215.283) (width 0.25) (layer "B.Cu") (net 2))
   (segment (start 214.3962 158.5162) (end 219.4762 158.5162) (width 0.25) (layer "B.Cu") (net 2))
   (segment (start 242.57 144.5514) (end 241.046 146.0754) (width 0.25) (layer "B.Cu") (net 2))
@@
   (segment (start 228.346 86.8426) (end 228.346 82.5246) (width 0.25) (layer "F.Cu") (net 3))
   (segment (start 228.346 82.5246) (end 231.394 82.5246) (width 0.25) (layer "F.Cu") (net 3))
-  (segment (start 288.417 70.739) (end 288.4028 70.7532) (width 0.25) (layer "F.Cu") (net 4))
-  (segment (start 288.4028 70.7532) (end 285.0408 70.7532) (width 0.25) (layer "F.Cu") (net 4))
+  (segment (start 288.29 70.7532) (end 285.0408 70.7532) (width 0.25) (layer "F.Cu") (net 4))
   (via (at 249.809 64.77) (size 0.8) (drill 0.4) (layers "F.Cu" "B.Cu") (net 4))
   (via (at 167.64 72.263) (size 0.8) (drill 0.4) (layers "F.Cu" "B.Cu") (net 4))
   (via (at 288.29 64.77) (size 0.8) (drill 0.4) (layers "F.Cu" "B.Cu") (net 4))
   (via (at 249.809 72.263) (size 0.8) (drill 0.4) (layers "F.Cu" "B.Cu") (net 4))
-  (via (at 288.417 70.739) (size 0.8) (drill 0.4) (layers "F.Cu" "B.Cu") (net 4))
+  (via (at 288.29 70.7532) (size 0.8) (drill 0.4) (layers "F.Cu" "B.Cu") (net 4))
   (segment (start 167.64 88.9) (end 167.64 72.263) (width 0.25) (layer "In1.Cu") (net 4))
+  (segment (start 288.29 70.7532) (end 288.29 64.77) (width 0.25) (layer "In1.Cu") (net 4))
   (segment (start 249.809 72.263) (end 249.809 64.77) (width 0.25) (layer "In1.Cu") (net 4))
   (segment (start 167.64 88.9) (end 167.64 93.7152) (width 0.25) (layer "In1.Cu") (net 4))
-  (segment (start 288.29 70.612) (end 288.417 70.739) (width 0.25) (layer "In1.Cu") (net 4))
-  (segment (start 288.29 64.77) (end 288.29 70.612) (width 0.25) (layer "In1.Cu") (net 4))
   (segment (start 167.64 72.263) (end 249.809 72.263) (width 0.25) (layer "In2.Cu") (net 4))
   (segment (start 249.809 64.77) (end 288.29 64.77) (width 0.25) (layer "In2.Cu") (net 4))

Commit message: 300 unrouted traces...
Routing:
- net Emulation: track 0.00 -> 117.1 mm, vias 0 -> 3
- net A0: track 61.9 -> 141.6 mm, vias 0 -> 2
- net A15: track 61.9 -> 120.2 mm, vias 0 -> 2
- net A14: track 62.6 -> 113.7 mm
- net A13: track 62.1 -> 109.9 mm
Changed lines of the file:
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@@
   (segment (start 259.2324 187.1218) (end 260.3574 188.2468) (width 0.25) (layer "In1.Cu") (net 61))
   (segment (start 260.3574 188.2468) (end 277.9702 188.2468) (width 0.25) (layer "In1.Cu") (net 61))
+  (via (at 168.402 153.035) (size 0.8) (drill 0.4) (layers "F.Cu" "B.Cu") (net 62))
+  (via (at 168.402 160.02) (size 0.8) (drill 0.4) (layers "F.Cu" "B.Cu") (net 62))
   (segment (start 239.395 189.7126) (end 240.52 190.8376) (width 0.25) (layer "In1.Cu") (net 62))
   (segment (start 221.1144 190.7614) (end 238.3462 190.7614) (width 0.25) (layer "In1.Cu") (net 62))
@@
   (segment (start 238.3462 190.7614) (end 239.395 189.7126) (width 0.25) (layer "In1.Cu") (net 62))
   (segment (start 260.3574 190.7868) (end 277.9702 190.7868) (width 0.25) (layer "In1.Cu") (net 62))
+  (segment (start 168.402 153.035) (end 168.402 160.02) (width 0.25) (layer "In1.Cu") (net 62))
   (segment (start 240.52 190.8376) (end 258.0566 190.8376) (width 0.25) (layer "In1.Cu") (net 62))
+  (segment (start 155.946 153.035) (end 168.402 153.035) (width 0.25) (layer "In2.Cu") (net 62))
+  (segment (start 168.402 160.02) (end 203.2 160.02) (width 0.25) (layer "In2.Cu") (net 62))
+  (segment (start 153.0554 150.1444) (end 155.946 153.035) (width 0.25) (layer "In2.Cu") (net 62))
   (segment (start 273.0574 193.6168) (end 274.4724 192.2018) (width 0.25) (layer "In2.Cu") (net 63))
   (segment (start 274.4724 192.2018) (end 275.9128 193.6422) (width 0.25) (layer "In2.Cu") (net 63))
   (segment (start 275.9128 193.6422) (end 292.8948 193.6422) (width 0.25) (layer "In2.Cu") (net 63))
+  (segment (start 154.2748 153.9038) (end 153.0554 152.6844) (width 0.25) (layer "In2.Cu") (net 63))
   (segment (start 235.2294 192.1764) (end 236.7206 193.6676) (width 0.25) (layer "In2.Cu") (net 63))
   (segment (start 292.8948 193.6422) (end 294.3098 192.2272) (width 0.25) (layer "In2.Cu") (net 63))
   (segment (start 253.22 193.6676) (end 254.635 192.2526) (width 0.25) (layer "In2.Cu") (net 63))
   (segment (start 255.9992 193.6168) (end 273.0574 193.6168) (width 0.25) (layer "In2.Cu") (net 63))
+  (segment (start 202.1638 153.9038) (end 154.2748 153.9038) (width 0.25) (layer "In2.Cu") (net 63))
   (segment (start 254.635 192.2526) (end 255.9992 193.6168) (width 0.25) (layer "In2.Cu") (net 63))
+  (segment (start 203.2 154.94) (end 202.1638 153.9038) (width 0.25) (layer "In2.Cu") (net 63))
   (segment (start 236.7206 193.6676) (end 253.22 193.6676) (width 0.25) (layer "In2.Cu") (net 63))
   (segment (start 273.3474 195.8668) (end 255.7092 195.8668) (width 0.25) (layer "In2.Cu") (net 64))
+  (segment (start 153.3398 154.94) (end 153.0554 155.2244) (width 0.25) (layer "In2.Cu") (net 64))
+  (segment (start 200.66 154.94) (end 153.3398 154.94) (width 0.25) (layer "In2.Cu") (net 64))
   (segment (start 253.51 195.9176) (end 236.4306 195.9176) (width 0.25) (layer "In2.Cu") (net 64))
   (segment (start 275.9128 196.1822) (end 274.4724 194.7418) (width 0.25) (layer "In2.Cu") (net 64))
@@
   (segment (start 258.0566 211.1576) (end 259.2324 209.9818) (width 0.25) (layer "In1.Cu") (net 76))
   (segment (start 260.3574 211.1068) (end 277.9702 211.1068) (width 0.25) (layer "In1.Cu") (net 76))
+  (via (at 114.173 183.388) (size 0.8) (drill 0.4) (layers "F.Cu" "B.Cu") (net 77))
+  (via (at 114.173 132.461) (size 0.8) (drill 0.4) (layers "F.Cu" "B.Cu") (net 77))
   (segment (start 219.9894 212.4964) (end 221.1144 213.6214) (width 0.25) (layer "In1.Cu") (net 77))
   (segment (start 259.2324 212.5218) (end 260.3574 213.6468) (width 0.25) (layer "In1.Cu") (net 77))
+  (segment (start 114.173 132.461) (end 114.173 183.388) (width 0.25) (layer "In1.Cu") (net 77))
   (segment (start 240.52 213.6976) (end 258.0566 213.6976) (width 0.25) (layer "In1.Cu") (net 77))
   (segment (start 277.9702 213.6468) (end 279.0698 212.5472) (width 0.25) (layer "In1.Cu") (net 77))
@@
   (segment (start 260.3574 213.6468) (end 277.9702 213.6468) (width 0.25) (layer "In1.Cu") (net 77))
   (segment (start 239.395 212.5726) (end 240.52 213.6976) (width 0.25) (layer "In1.Cu") (net 77))
+  (segment (start 135.5932 130.1422) (end 116.4918 130.1422) (width 0.25) (layer "In2.Cu") (net 77))
+  (segment (start 137.8154 132.3644) (end 135.5932 130.1422) (width 0.25) (layer "In2.Cu") (net 77))
+  (segment (start 114.173 183.388) (end 114.2188 183.3422) (width 0.25) (layer "In2.Cu") (net 77))
+  (segment (start 114.2188 183.3422) (end 117.47 183.3422) (width 0.25) (layer "In2.Cu") (net 77))
+  (segment (start 116.4918 130.1422) (end 114.173 132.461) (width 0.25) (layer "In2.Cu") (net 77))
   (via (at 278.511 172.974) (size 0.8) (drill 0.4) (layers "F.Cu" "B.Cu") (net 79))
   (segment (start 278.511 172.974) (end 278.4856 172.9486) (width 0.25) (layer "In1.Cu") (net 79))
@@
   (segment (start 140.97 174.879) (end 139.319 174.879) (width 0.25) (layer "In2.Cu") (net 169))
   (segment (start 141.0004 129.8244) (end 153.0554 129.8244) (width 0.25) (layer "In2.Cu") (net 169))
+  (via (at 176.657 124.714) (size 0.8) (drill 0.4) (layers "F.Cu" "B.Cu") (net 171))
+  (via (at 176.784 164.719) (size 0.8) (drill 0.4) (layers "F.Cu" "B.Cu") (net 171))
+  (via (at 222.377 164.719) (size 0.8) (drill 0.4) (layers "F.Cu" "B.Cu") (net 171))
+  (segment (start 176.657 124.714) (end 176.657 164.592) (width 0.25) (layer "In1.Cu") (net 171))
+  (segment (start 222.377 164.719) (end 222.377 158.877) (width 0.25) (layer "In1.Cu") (net 171))
+  (segment (start 222.377 158.877) (end 220.98 157.48) (width 0.25) (layer "In1.Cu") (net 171))
+  (segment (start 176.657 164.592) (end 176.784 164.719) (width 0.25) (layer "In1.Cu") (net 171))
+  (segment (start 176.6266 124.7444) (end 176.657 124.714) (width 0.25) (layer "In2.Cu") (net 171))
+  (segment (start 176.784 164.719) (end 222.377 164.719) (width 0.25) (layer "In2.Cu") (net 171))
+  (segment (start 153.0554 124.7444) (end 176.6266 124.7444) (width 0.25) (layer "In2.Cu") (net 171))
   (via (at 223.52 172.339) (size 0.8) (drill 0.4) (layers "F.Cu" "B.Cu") (net 179))
   (segment (start 223.52 172.339) (end 223.52 160.02) (width 0.25) (layer "In1.Cu") (net 179))

Commit message: 288 unrouted traces...
Routing:
- net RESET: track 0.00 -> 134.1 mm, vias 0 -> 5
- net ~{WRITE}: track 61.9 -> 153.0 mm, vias 0 -> 5
- net IDE_D15: track 0.00 -> 88.8 mm, vias 0 -> 2
- net A2: track 62.1 -> 145.0 mm, vias 0 -> 2
- net IDE_D14: track 0.00 -> 81.2 mm, vias 0 -> 2
- net A1: track 61.9 -> 142.2 mm, vias 0 -> 2
- net R/~{W}: track 0.00 -> 75.1 mm, vias 0 -> 3
- net IDE_D13: track 0.00 -> 73.6 mm, vias 0 -> 2
- net IDE_D12: track 0.00 -> 66.0 mm, vias 0 -> 2
- net D0: track 99.9 -> 162.7 mm, vias 2 -> 6
- net +5V: track 930.9 -> 945.9 mm, vias 11 -> 12

Commit message: 268 unrouted traces...
Routing:
- net CLK_STR: track 24.4 -> 205.6 mm, vias 0 -> 3
- net ~{ABORT}: track 0.00 -> 169.9 mm, vias 0 -> 6
- net BusEnable: track 0.00 -> 162.4 mm, vias 0 -> 3
- net ~{FLASH4_EN}: track 0.00 -> 145.3 mm, vias 0 -> 5
- net ~{NMI}: track 34.1 -> 172.3 mm, vias 1 -> 6
- net R/~{W}: track 75.1 -> 213.1 mm, vias 3 -> 4
- net VPA: track 0.00 -> 135.0 mm, vias 0 -> 3
- net ~{RAM0_EN}: track 0.00 -> 120.2 mm, vias 0 -> 4
- net A3: track 61.9 -> 171.5 mm, vias 0 -> 3
- net ~{WRITE}: track 153.0 -> 256.3 mm, vias 5 -> 8
- net ~{IRQ}: track 24.0 -> 123.4 mm, vias 1 -> 3
- net Net-(JP1-C): track 0.00 -> 72.1 mm, vias 0 -> 2
- net A4: track 61.9 -> 131.0 mm, vias 0 -> 2
- net GND: track 1222.1 -> 1289.0 mm, vias 4 -> 5
- net D7: track 62.1 -> 105.9 mm, vias 0 -> 2
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
Commit message: 268 unrouted traces...
Parts:
- added U19: GAL16V8, Package_DIP:DIP-20_W7.62mm_Socket_LongPads, F.Cu at (305.4, 117.1)
Routing:
- net ~{IDE_CS0}: track 0.00 -> 92.4 mm, vias 0 -> 2
- net ~{IDE_CS1}: track 0.00 -> 90.5 mm, vias 0 -> 2
- net ~{IDE_WRITE}: track 0.00 -> 67.0 mm, vias 0 -> 2
- net ~{WRITE}: track 256.3 -> 304.0 mm, vias 8 -> 10
- net IDE_CS0: track 0.00 -> 29.5 mm, vias 0 -> 1
- net IDE_READ: track 0.00 -> 12.2 mm
- net IDE_WRITE: track 0.00 -> 11.7 mm
- net IDE_RESET: track 0.00 -> 11.7 mm
- net IDE_CS1: track 0.00 -> 11.7 mm
- net GND: track 1289.0 -> 1295.9 mm
- net +5V: track 945.9 -> 951.7 mm

Commit message: 268 unrouted traces...
Parts:
- added REF**: KiCad-Logo2_5mm_SilkScreen, Symbol:KiCad-Logo2_5mm_SilkScreen, F.Cu at (92.1, 165.5)
- added REF**: OSHW-Logo_5.7x6mm_SilkScreen, Symbol:OSHW-Logo_5.7x6mm_SilkScreen, F.Cu at (97.3, 158.9)

Commit message: 265 unrouted traces...
Parts:
- removed REF**: KiCad-Logo2_5mm_SilkScreen, Symbol:KiCad-Logo2_5mm_SilkScreen
- removed REF**: OSHW-Logo_5.7x6mm_SilkScreen, Symbol:OSHW-Logo_5.7x6mm_SilkScreen
Routing:
- net VDA: track 0.00 -> 133.2 mm, vias 0 -> 3
- net ~{IRQ}: track 123.4 -> 216.9 mm, vias 3 -> 5
- net ~{FLASH2_EN}: track 0.00 -> 78.6 mm, vias 0 -> 3

Commit message: 260 unrouted traces...
Routing:
- net ~{HALT}: track 135.1 -> 233.0 mm, vias 2 -> 4
- net A9: track 149.8 -> 210.3 mm, vias 3 -> 5
- net A15: track 120.2 -> 166.4 mm, vias 2 -> 3
- net ~{RAM0_EN}: track 120.2 -> 161.6 mm, vias 4 -> 7
- net D0: track 162.7 -> 192.9 mm, vias 6 -> 8
